Commit message: Update URDF paths

File: urdf/biotac/shell_core/biotac.urdf (robot description, URDF)
Before this commit: robot biotac, 2 links, 1 joints
Links:
- link bc: geometry collision mesh filename=../../../meshes/biotac/bc/top_side_core_bc.obj; visual mesh filename=../../../meshes/biotac/bc/top_side_core_bc.obj

File: urdf/biotac/shell_core/biotac_template.urdf (robot description, URDF)
Before this commit: robot biotac, 2 links, 1 joints
Links:
- link bc: geometry collision mesh filename=../../../meshes/biotac/bc/top_side_core_bc.obj; visual mesh filename=../../../meshes/biotac/bc/top_side_core_bc.obj
